File: hardware/INTech - Carte de Base/INTech - Carte de Base.sch (EAGLE design)
At the start: 41 parts

Commit message: Ajout de texte pour les régulateurs de tension
Parts:
- DC1: value R-78C5.0-1.0 -> R-78C-1.0_INTECH; device dc-dc-converter:R-78C5.0-1.0 -> dc-dc-converter:R-78C-1.0_INTECH
Other:
- moved on the sheet: DC1
Changed lines of the file:
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@@
 <setting verticaltext="up"/>
 </settings>
-<grid distance="0.1" unitdist="inch" unit="inch" style="lines" multiple="1" display="no" altdistance="0.01" altunitdist="inch" altunit="inch"/>
+<grid distance="0.1" unitdist="inch" unit="inch" style="lines" multiple="1" display="yes" altdistance="0.01" altunitdist="inch" altunit="inch"/>
 <layers>
 <layer number="1" name="Top" color="4" fill="1" visible="no" active="no"/>
@@
 <part name="C12" library="resistor" deviceset="CPOL-EU" device="E2.5-6" value="22µF"/>
 <part name="L1" library="inductor-neosid" deviceset="SD12" device="K100" value="68µH"/>
-<part name="DC1" library="dc-dc-converter" deviceset="R-78C*-1.0" device="" technology="5.0"/>
+<part name="DC1" library="dc-dc-converter" deviceset="R-78C*-1.0_INTECH" device=""/>
 <part name="DEL_RASP" library="con-ptr500" deviceset="AK300/2" device=""/>
 <part name="USB_RASP" library="con-berg" deviceset="PN87520" device=""/>

Commit message: Légères modif et ajout de 2 librairies
Parts:
- USB_RASP: value (none) -> USB_87520; device con-berg:PN87520 -> USB_CF_INTech:USB_87520
Connections:
- net +5V_RASP: now also USB_RASP.VIN; no longer USB_RASP.1
- net GND: now also USB_RASP.GND; no longer USB_RASP.4
Other:
- moved on the sheet: AX-12-EXEMPLE, USB_RASP
Changed lines of the file:
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@@
 <setting verticaltext="up"/>
 </settings>
-<grid distance="0.1" unitdist="inch" unit="inch" style="lines" multiple="1" display="yes" altdistance="0.01" altunitdist="inch" altunit="inch"/>
+<grid distance="0.1" unitdist="inch" unit="inch" style="lines" multiple="1" display="no" altdistance="0.01" altunitdist="inch" altunit="inch"/>
 <layers>
 <layer number="1" name="Top" color="4" fill="1" visible="no" active="no"/>
@@
 <part name="DC1" library="dc-dc-converter" deviceset="R-78C*-1.0_INTECH" device=""/>
 <part name="DEL_RASP" library="con-ptr500" deviceset="AK300/2" device=""/>
-<part name="USB_RASP" library="con-berg" deviceset="PN87520" device=""/>
+<part name="USB_RASP" library="USB_CF_INTech" deviceset="USB_87520" device=""/>
 </parts>
 <sheets>
@@
 <junction x="-215.9" y="-121.92"/>
 <wire x1="-215.9" y1="-124.46" x2="-215.9" y2="-121.92" width="0.1524" layer="91"/>
-<pinref part="USB_RASP" gate="G$1" pin="4"/>
+<pinref part="USB_RASP" gate="G$1" pin="GND"/>
 <junction x="-185.42" y="-124.46"/>
 <wire x1="-215.9" y1="-124.46" x2="-185.42" y2="-124.46" width="0.1524" layer="91"/>
@@
 <net name="+5V_RASP" class="0">
 <segment>
-<pinref part="USB_RASP" gate="G$1" pin="1"/>
+<pinref part="USB_RASP" gate="G$1" pin="VIN"/>
 <junction x="-185.42" y="-116.84"/>
 <wire x1="-185.42" y1="-116.84" x2="-185.42" y2="-114.3" width="0.1524" layer="91"/>
